File: hardware/ai_glasses_carrier.kicad_sch (KiCad schematic)
At the start: 102 parts, among them J1 DF40C-100DS-0.4V(51), J2 FH35C-31S-0.3SHW(50), J3 JST-SH 2p (spkr), J31 DF40C-100DS-0.4V(51), J32 DF40C-100DS-0.4V(51), J4 GCT USB4085 (USB2), J5 JST-PH 3p, J6 JST-SH 2p, J7 Header 1x4 2.54mm, J8 U.FL / IPEX, SW1 Tact SW SMD, SW2 Tact SW SMD, SW3 Tact SW SMD, U10 ICM-42688-P, U11 DRV2605L, U12 TLV75733 (LDO), U13 TLV75718 (LDO), U14 MAX-M10S-00B-01, U15 TPS25940 (e-fuse, opt), U16 TPD4E05U06, U2 TPD4E05U06, U3 LP5907-3.3 (low-noise LDO), U4 MAX98357AETE+T, U5 TPD2E009, U6 TPS61022 (Boost), U7 BQ25180, U8 BQ29700, U9 MAX17048

Commit message: Update V2 chipdown schematic and mechanical package
Parts:
- D4: footprint AI_Glasses:RF_ESD_2P_VERIFY -> Diode_SMD:D_SOD-882
- J1: footprint AI_Glasses:VERIFY_B2B_J1_LOGICAL -> Connector_Hirose_DF40:Hirose_DF40C-100DS-0.4V_2x50_P0.4mm
- J3, J6: footprint AI_Glasses:VERIFY_2P -> Connector_JST:JST_SH_BM02B-SRSS-TB_1x02-1MP_P1.00mm_Vertical
- J31: footprint AI_Glasses:VERIFY_B2B_J31_LOGICAL -> Connector_Hirose_DF40:Hirose_DF40C-100DS-0.4V_2x50_P0.4mm
- J32: footprint AI_Glasses:VERIFY_B2B_J32_LOGICAL -> Connector_Hirose_DF40:Hirose_DF40C-100DS-0.4V_2x50_P0.4mm
- J4: footprint AI_Glasses:VERIFY_7P -> Connector_USB:USB_C_Receptacle_GCT_USB4085
- J5: footprint AI_Glasses:VERIFY_3P -> Connector_JST:JST_PH_S3B-PH-SM4-TB_1x03-1MP_P2.00mm_Horizontal
- J8: footprint AI_Glasses:VERIFY_2P -> Connector_Coaxial:U.FL_Hirose_U.FL-R-SMT-1_Vertical
- MK1, MK2: footprint AI_Glasses:VERIFY_5P -> Sensor_Audio:Knowles_LGA-5_3.5x2.65mm
- SW1, SW2, SW3: footprint AI_Glasses:VERIFY_2P -> Button_Switch_SMD:SW_Push_1P1T_NO_CK_KMR2
- TP1, TP10, TP11, TP12, TP13, TP14, TP15, TP16, TP2, TP3, TP4, TP5, TP6, TP7, TP8, TP9: footprint AI_Glasses:VERIFY_TP_1P -> TestPoint:TestPoint_Pad_D1.5mm
- U10: footprint AI_Glasses:VERIFY_5P -> Package_LGA:LGA-14_3x2.5mm_P0.5mm_LayoutBorder3x4y
- U11: footprint AI_Glasses:VERIFY_6P -> Package_SO:MSOP-10_3x3mm_P0.5mm
- U12, U13, U8: footprint AI_Glasses:VERIFY_3P -> Package_TO_SOT_SMD:SOT-23-5
- U14: footprint AI_Glasses:VERIFY_9P -> RF_GPS:ublox_MAX
- U15: footprint AI_Glasses:VERIFY_4P -> Package_DFN_QFN:Texas_RGP0020H_VQFN-20-1EP_4x4mm_P0.5mm_EP2.4x2.4mm
- U16, U2: footprint AI_Glasses:TPD4E05U06_VERIFY -> Package_SON:USON-10_2.5x1.0mm_P0.5mm
- U3: footprint AI_Glasses:VERIFY_4P -> Package_TO_SOT_SMD:SOT-23-5
- U4: footprint AI_Glasses:VERIFY_9P -> Package_DFN_QFN:QFN-16-1EP_3x3mm_P0.5mm_EP1.45x1.45mm
- U5: footprint AI_Glasses:TPD2E009_VERIFY -> Package_TO_SOT_SMD:SOT-553
- U6: footprint AI_Glasses:VERIFY_5P -> Package_DFN_QFN:Texas_RWU0007A_VQFN-7_2x2mm_P0.5mm
- U7: footprint AI_Glasses:VERIFY_8P -> Package_BGA:Texas_DSBGA-12_1.36x1.86mm_Layout3x4_P0.5mm
- U9: footprint AI_Glasses:VERIFY_6P -> Package_DFN_QFN:DFN-8-1EP_2x3mm_P0.5mm_EP0.61x2.2mm
