File: v2_chipdown/hardware/ai_glasses_v2_chipdown.kicad_sch (KiCad schematic)
At the start: 96 parts, among them J1 Magnetic pogo 4-6p, J2 USB-C 16p USB2-only, J3 Hirose FH26W 0.3mm FPC, J4 Custom hinge FPC 6-10mm, J5 U.FL / I-PEX MHF, J6 BLE 2.4 GHz FPC/PCB ant, J7 Wi-Fi 2.4/5 GHz FPC ant, M1 LRA/ERM motor, Q1 Dual N-MOSFET (b2b), SW1 Power/PWRKEY, SW2 Reset, SW3 MaskROM/Recovery, U1 RK3576, U10 BMI270, U11 FCU760KAAMD, U12 TPS62825, U13 TPS22917DBVR, U14 IMX415-AAQR module (custom FP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, U15 TPS62840, U16 TLV75529PDRVR, U17 TPS22917DBVR, U18 TPD4E05U06, U19 TPD4E05U06, U2 RK806S-5, U20 MAX98360A, U21 TPS22917DBVR, U22 DRV2605L, U23 BQ2970, U24 TPD2E001, U25 INA238 (I_BAT_TOTAL), U26 INA238 (I_CELL_L), U27 INA238 (I_CELL_R), U28 INA238 (I_SOC_5V), U29 INA238 (I_WIFI), U3 LPDDR4X 4GB (MPN TBD), U30 INA238 (I_AUDIO), U31 INA238 (I_CAM_1V1), U32 INA238 (I_CAM_1V8), U33 INA238 (I_CAM_2V9), U4 eMMC 5.1 32GB (MPN TBD), U5 MX25U6432F, U6 TPS61088, U7 nRF54L15-QFN48, U8 nPM1300, U9 NDP120, Y1 24 MHz 10 ppm XTAL

Commit message: Update V2 chipdown schematic and mechanical package
Parts:
- removed C2: 0.1uF, symbol aiglassesv2:C2
- removed J4: Custom hinge FPC 6-10mm, symbol aiglassesv2:J4
- removed Q1: Dual N-MOSFET (b2b), symbol aiglassesv2:Q1
- removed R11: 100k, symbol aiglassesv2:R11
- removed R13: 100k, symbol aiglassesv2:R13
- removed R14: 100k, symbol aiglassesv2:R14
- removed R15: 100k, symbol aiglassesv2:R15
- removed R16: 100k, symbol aiglassesv2:R16
- removed R17: 100k, symbol aiglassesv2:R17
- removed R21: 0R (pack-PCM baseline), symbol aiglassesv2:R21
- removed R22: 330R, symbol aiglassesv2:R22
- removed R23: 2k, symbol aiglassesv2:R23
- removed RS2: 10 mohm 1%, symbol aiglassesv2:RS2
- removed SW1: Power/PWRKEY, symbol aiglassesv2:SW1
- removed SW2: Reset, symbol aiglassesv2:SW2
- removed U16: TLV75529PDRVR, symbol aiglassesv2:U16
- removed U17: TPS22917DBVR, symbol aiglassesv2:U17
- removed U23: BQ2970, symbol aiglassesv2:U23
- removed U31: INA238 (I_CAM_1V1), symbol aiglassesv2:U31
- removed U4: eMMC 5.1 32GB (MPN TBD), symbol aiglassesv2:U4
- removed U8: nPM1300, symbol aiglassesv2:U8
- added MK3: T5837 (array mic 2), symbol aiglassesv2:MK3
- added MK4: T5837 (4th mic), symbol aiglassesv2:MK4
- added PCM1: Supplier 1S2P pack PCM + protection FETs, symbol aiglassesv2:PCM1
- added R10: 2.2k 1%, symbol aiglassesv2:R10
- added R20: 100k, symbol aiglassesv2:R20
- added R3: 2.2k 1%, symbol aiglassesv2:R3
- added R4: 2.2k 1%, symbol aiglassesv2:R4
- added R5: 2.2k 1%, symbol aiglassesv2:R5
- added R6: 2.2k 1%, symbol aiglassesv2:R6
- added R9: 2.2k 1%, symbol aiglassesv2:R9
- added RS9: 100 mohm 1%, symbol aiglassesv2:RS9
- added TP2: Battery test points, symbol aiglassesv2:TP2
- added U10: BMI270, symbol aiglassesv2:U10
- added U27: INA238 (I_CELL_R), symbol aiglassesv2:U27
- added U34: TPD4E05U06, symbol aiglassesv2:U34
- added U35: BQ25895, symbol aiglassesv2:U35
- added U36: 5V input eFuse/OVP (MPN TBD), symbol aiglassesv2:U36
- added Y1: 24 MHz 10 ppm XTAL, symbol aiglassesv2:Y1
- J1: value Magnetic pogo 4-6p -> CCP P2578MP01-06C180HT; Assembly TBD -> HOLD; Gate Magnet direction, sweat corrosion, short, cycle life -> USB2 eye/contact validation, current/fault/ESD, mating STEP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; Package AI_Glasses_V2:VERIFY_POGO -> AI_Glasses_V2:VERIFY_POGO_6P_1.8MM
- J3: value Hirose FH26W 0.3mm FPC -> Hirose FH26W-33S-0.3SHW(97); Gate G12 (pin count from final cam lane/mic/power split) -> G10/G12 (camera module vendor signs 33-pin pinout, contact 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; Package AI_Glasses_V2:VERIFY_FPC_FH26W -> AI_Glasses_V2:VERIFY_FH26W_33S_0.3SHW
- J5: value U.FL / I-PEX MHF -> U.FL / I-PEX MHF RF test connector; Assembly Fit -> DNP; Gate Connector height + mating life -> EVT RF debug only; production prefers direct coax or solder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; now not fitted
- J6: value BLE 2.4 GHz FPC/PCB ant -> FCU760K ANT_BT DNP test pad; Assembly TBD -> DNP; Gate Worn-state tuning; clear of battery/metal -> Only populate if Quectel FAE + coexistence test requires th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; now not fitted
- J7: value Wi-Fi 2.4/5 GHz FPC ant -> Taoglas FXP840.07.0055B; Assembly TBD -> HOLD; Gate Head-loaded RSSI/throughput/SAR; keep-out -> G14 (worn-state tune + antenna keep-out in full shell with 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; Package AI_Glasses_V2:VERIFY_ANT -> AI_Glasses_V2:VERIFY_FPC_ANT_14x5
- L1: value Boost inductor (TBD) -> Coilcraft XGL4020-102MEC 1.0uH; Assembly TBD -> HOLD; Gate G06/G13 (Isat covers boot+AI peak; height <=2mm; thermal) -> G06/G13 (Isat/DCR/thermal pass for 5.1V 3A continuous / 4A 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; Package AI_Glasses_V2:VERIFY_L_5x5 -> AI_Glasses_V2:VERIFY_L_4x4x2_XGL4020
- LS1: value 8 ohm 0.5-1 W speaker -> CUI CMS-15113-078SP-67; Assembly TBD -> HOLD; Gate MPN after acoustic cavity/volume/leak test -> Acoustic EVT: 0.3-0.5cc cavity, port/foam seal, magnet-to-a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; Package AI_Glasses_V2:VERIFY_SPK -> AI_Glasses_V2:VERIFY_SPK_15x11x3
- R11: renamed from R18; symbol aiglassesv2:R18 -> aiglassesv2:R11; BOM_ID C046h -> C046a; Gate Default OFF (§4/§9: FCU760K CHIP_EN default low) -> Default OFF (§4)
- R12: renamed from R19; symbol aiglassesv2:R19 -> aiglassesv2:R12; BOM_ID C046i -> C046b
- R13: renamed from R20; symbol aiglassesv2:R20 -> aiglassesv2:R13; BOM_ID C046j -> C046c; Board R-Temple Compute Board -> Front Sensor Board
- R14: renamed from R3; value 2.2k 1% -> 100k; symbol aiglassesv2:R3 -> aiglassesv2:R14; BOM_ID C045a -> C046d; Board L-Temple AON/Power Board -> Front Sensor Board; Gate Confirm vs total AON bus capacitance -> Default OFF (§4)
- R15: renamed from R4; value 2.2k 1% -> 100k; symbol aiglassesv2:R4 -> aiglassesv2:R15; BOM_ID C045b -> C046e; Board L-Temple AON/Power Board -> Front Sensor Board; Gate Confirm vs total AON bus capacitance -> Default OFF (§4)
- R16: renamed from R5; value 2.2k 1% -> 100k; symbol aiglassesv2:R5 -> aiglassesv2:R16; BOM_ID C045c -> C046f; Board Front Sensor Board -> R-Temple Compute Board; Gate Confirm vs camera bus capacitance -> Default OFF (§4)
- R17: renamed from R6; value 2.2k 1% -> 100k; symbol aiglassesv2:R6 -> aiglassesv2:R17; BOM_ID C045d -> C046g; Board Front Sensor Board -> R-Temple Compute Board; Gate Confirm vs camera bus capacitance -> Default OFF (§4)
- R18: renamed from R9; value 2.2k 1% -> 100k; symbol aiglassesv2:R9 -> aiglassesv2:R18; BOM_ID C045e -> C046h; Gate Confirm vs SoC PMIC bus -> Default OFF (§4/§9: FCU760K CHIP_EN default low)
- R19: renamed from R10; value 2.2k 1% -> 100k; symbol aiglassesv2:R10 -> aiglassesv2:R19; BOM_ID C045f -> C046i; Gate Confirm vs SoC PMIC bus -> Default OFF (§4)
- RS2: renamed from TP2; value Battery test points -> 10 mohm 1%; symbol aiglassesv2:TP2 -> aiglassesv2:RS2; BOM_ID C033-TP -> C044-RCL; Gate Cell/pack voltage + NTC probe access (§21) -> Branch current-share (§7/§29); Package AI_Glasses_V2:TestPad_Set -> AI_Glasses_V2:R_0805_shunt
- RS8: renamed from U27; value INA238 (I_CELL_R) -> 100 mohm 1%; symbol aiglassesv2:U27 -> aiglassesv2:RS8; Assembly DNP -> Fit; BOM_ID C044-ICR -> C044-RC8; Board Temple Rears (batt/spkr/ant) -> Front Sensor Board; Gate Power Gate — EVT-A only (current-share) -> Per-rail Kelvin (§23/§29); IOVDD ~3mA; Package AI_Glasses_V2:VSSOP-10 -> AI_Glasses_V2:R_0402_shunt; Priority P1 -> P0; now fitted
- RT1: value 10k NTC (R cell) -> 10k NTC B=3435 1% (R cell); Gate NTC curve matched to nPM1300 charger config -> NTC curve/package/placement matched to pack supplier + BQ25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
- RT2: value 10k NTC (L cell) -> 10k NTC B=3435 1% (L cell); Gate NTC curve matched to nPM1300 charger config -> NTC curve/package/placement matched to pack supplier + ADC/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
- SW1: renamed from RS8; value 100 mohm 1% -> Power/PWRKEY; symbol aiglassesv2:RS8 -> aiglassesv2:SW1; BOM_ID C044-RC8 -> C042a; Board Front Sensor Board -> EVT Debug Tail; Gate Per-rail Kelvin (§23/§29); IOVDD ~3mA -> First chip-down must recover from boot failure; Package AI_Glasses_V2:R_0402_shunt -> Button_Switch_SMD:SW_Push_1P1T_NO_CK_KMR2
- SW2: renamed from RS9; value 100 mohm 1% -> Reset; symbol aiglassesv2:RS9 -> aiglassesv2:SW2; BOM_ID C044-RC29 -> C042b; Board Front Sensor Board -> EVT Debug Tail; Gate Per-rail Kelvin (§23/§29); AVDD ~156mA -> Bring-up; Package AI_Glasses_V2:R_0603_shunt -> Button_Switch_SMD:SW_Push_1P1T_NO_CK_KMR2
- U14: value IMX415-AAQR module (custom FPC) -> Sony IMX415-AAQR-C custom module
- U16: renamed from MK3; value T5837 (array mic 2) -> TLV75529PDRVR; symbol aiglassesv2:MK3 -> aiglassesv2:U16; BOM_ID C013c -> C021; Gate G11 -> Verify vs IMX415 AVDD peak (156mA) + PSRR; Package AI_Glasses_V2:LGA-5_3.5x2.65 -> AI_Glasses_V2:WSON-6_2x2
- U17: renamed from MK4; value T5837 (4th mic) -> TPS22917DBVR; symbol aiglassesv2:MK4 -> aiglassesv2:U17; Assembly DNP -> Fit; BOM_ID C014 -> C022; Gate G11 (populate only if array sim/proto needs it) -> Check reverse block, ramp, QOD, logic level; Package AI_Glasses_V2:LGA-5_3.5x2.65 -> Package_TO_SOT_SMD:SOT-23-5; Priority P1 -> P0; now fitted
- U2: value RK806S-5 -> RK806S-5 QFN68 7x7x0.90mm; Gate G03 (RK806S MPN/inductors/caps/timing per Radxa/Rockchip FA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 -> G03 (official RK806S-5 datasheet, OTP/default rails, sequen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; Package AI_Glasses_V2:VERIFY_QFN -> AI_Glasses_V2:VERIFY_QFN68_7x7_EP5.49_P0.35
- U3: value LPDDR4X 4GB (MPN TBD) -> Samsung K4U6E3S4AA-MGCL; Gate G02 (LPDDR4X MPN/topology/placement, DDR review + length re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 -> G02 (Samsung datasheet/ball map/IBIS + Rockchip DDR AVL/ini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; Package AI_Glasses_V2:VERIFY_BGA -> AI_Glasses_V2:VERIFY_FBGA200_0.65
- U31: renamed from R12; value 100k -> INA238 (I_CAM_1V1); symbol aiglassesv2:R12 -> aiglassesv2:U31; Assembly Fit -> DNP; BOM_ID C046b -> C044-IC1; Board R-Temple Compute Board -> Front Sensor Board; Gate Default OFF (§4) -> Power Gate — EVT-A only; Package AI_Glasses_V2:R_0402 -> AI_Glasses_V2:VSSOP-10; Priority P0 -> P1; now not fitted
- U4: renamed from Y1; value 24 MHz 10 ppm XTAL -> Samsung KLMAG1JENB-B041; symbol aiglassesv2:Y1 -> aiglassesv2:U4; Assembly Fit -> HOLD; BOM_ID C005 -> C004; Gate G01 (reuse reference CL/ESR + placement distance per HDG) -> G04 (official Samsung datasheet/package + BSP boot/HS200 th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; Package AI_Glasses_V2:Crystal_SMD_3225 -> AI_Glasses_V2:VERIFY_BGA153
- U8: renamed from U10; value BMI270 -> nPM1300; symbol aiglassesv2:U10 -> aiglassesv2:U8; Assembly Fit -> HOLD; BOM_ID C012 -> C010; Gate Evaluate false-trigger under real frame vibration -> G08 (AON <=25/50mW) — configure via nPM PowerUP on EK befor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; Package Package_LGA:LGA-14_2.5x3mm_P0.5mm -> AI_Glasses_V2:QFN_5x5
Connections:
- net AON_1V8: now also U17.1 (VIN), U8.5 (BUCK1), R3.1 (A), R4.1 (A), U10.1 (VDD), U10.2 (VDDIO); no longer J3.18 (AON_1V8), R14.1 (A), R15.1 (A), U8.1 (VDD), U8.2 (VDDIO)
- net AON_3V3: now also U8.6 (BUCK2), MK3.1 (VDD); no longer J3.19 (AON_3V3), U16.1 (VDD)
- net AON_LSW2: now also U8.7 (LSW2), MK4.1 (VDD); no longer U17.1 (VDD)
- net AUDIO_AMP_SD: now also R20.1 (A); no longer R13.1 (A)
- net AUDIO_LS_EN: now also R19.1 (A); no longer R12.1 (A)
- net BATL_F: now also RS2.1 (A)
- net BATL_P: now also TP2.1 (CELL_L); no longer RS2.1 (CELL_L)
- net BATR_F: now also U27.1 (IN_P); no longer RS8.1 (IN_P)
- net BATR_P: now also TP2.2 (CELL_R); no longer RS2.2 (CELL_R)
- net BAT_P: now also RS2.2 (B), PCM1.1 (PACK_PLUS), TP2.3 (PACK_P), U27.2 (IN_N); no longer RS2.3 (PACK_P), RS8.2 (IN_N)
- net BLE_ANT: now also U11.12 (ANT_BT_DNP); no longer U7.4 (ANT)
- net CAM_1V1: now also U31.1 (IN_P)
- net CAM_1V1_EN: now also R13.1 (A); no longer J3.21 (CAM_1V1_EN)
- net CAM_1V1_S: now also J3.2 (2_DVDD), U31.2 (IN_N)
- net CAM_1V8_EN: now also R14.1 (A), U17.3 (EN); no longer J3.22 (CAM_1V8_EN)
- net CAM_1V8_S: now also J3.6 (6_IOVDD), RS8.2 (B); no longer SW1.2 (B)
- net CAM_1V8_SW: now also RS8.1 (A), U17.2 (VOUT), R5.1 (A), R6.1 (A); no longer R16.1 (A), R17.1 (A), SW1.1 (A)
- net CAM_2V9: now also U16.4 (VOUT), RS9.1 (A); no longer SW2.1 (A)
- net CAM_2V9_EN: now also R15.1 (A), U16.2 (EN); no longer J3.23 (CAM_2V9_EN)
- net CAM_2V9_S: now also J3.4 (4_AVDD), RS9.2 (B); no longer SW2.2 (B)
- net CAM_I2C_SCL: now also J3.10 (10_I2C_SCL), U1.32 (CAM_I2C_SCL), U14.15 (SCL), R5.2 (B); no longer J3.7 (CAM_I2C_SCL), R16.2 (B), U1.28 (CAM_I2C_SCL), U14.11 (SCL)
- net CAM_I2C_SDA: now also J3.11 (11_I2C_SDA), U1.33 (CAM_I2C_SDA), U14.16 (SDA), R6.2 (B); no longer J3.8 (CAM_I2C_SDA), R17.2 (B), U1.29 (CAM_I2C_SDA), U14.12 (SDA)
- net CAM_MCLK: now also J3.8 (8_MCLK), U1.36 (CAM_MCLK), U14.19 (INCK); no longer J3.11 (CAM_MCLK), U1.32 (CAM_MCLK), U14.15 (INCK)
- net CAM_PWDN_L: now also J3.13 (13_PWDN), U1.35 (CAM_PWDN_L), U14.18 (PWDN_L); no longer J3.10 (CAM_PWDN_L), U1.31 (CAM_PWDN_L), U14.14 (PWDN_L)
- net CAM_RST_L: now also J3.12 (12_RESET_N), U1.34 (CAM_RST_L), U14.17 (XCLR_L); no longer J3.9 (CAM_RST_L), U1.30 (CAM_RST_L), U14.13 (XCLR_L)
- net CELL_NEG: now also PCM1.3 (CELL_MINUS), TP2.4 (CELL_NEG); no longer RS2.4 (CELL_NEG)
- net CSI_CLK_N: now also J3.16 (16_MIPI_CLK_N); no longer J3.2 (CSI_CLK_N)
- net CSI_CLK_P: now also J3.17 (17_MIPI_CLK_P); no longer J3.1 (CSI_CLK_P)
- net CSI_D0_N: now also J3.19 (19_MIPI_D0_N); no longer J3.4 (CSI_D0_N)
- net CSI_D0_P: now also J3.20 (20_MIPI_D0_P); no longer J3.3 (CSI_D0_P)
- net CSI_D1_N: now also J3.22 (22_MIPI_D1_N); no longer J3.6 (CSI_D1_N)
- net CSI_D1_P: now also J3.23 (23_MIPI_D1_P); no longer J3.5 (CSI_D1_P)
- net DSP_FAULT: now also U7.38 (DSP_FAULT); no longer U7.34 (DSP_FAULT)
- net DSP_READY: now also U7.37 (DSP_READY); no longer U7.33 (DSP_READY)
- net DSP_RESET_L: now also U7.39 (DSP_RST_n); no longer U7.35 (DSP_RST_n)
- net DSP_SPI_CS_n: now also U7.35 (DSP_CS_n); no longer U7.31 (DSP_CS_n)
- net DSP_SPI_MISO: now also U7.34 (DSP_MISO); no longer U7.30 (DSP_MISO)
- net DSP_SPI_MOSI: now also U7.33 (DSP_MOSI); no longer U7.29 (DSP_MOSI)
- net DSP_SPI_SCK: now also U7.32 (DSP_SCK); no longer U7.28 (DSP_SCK)
- net DSP_WAKE: now also U7.36 (DSP_WAKE); no longer U7.32 (DSP_WAKE)
- net EMMC_BUS: now also U4.4 (EMMC_BUS)
- net GND: now also J1.1 (GND1), J1.4 (GND2), J3.1 (1_GND), J3.15 (15_GND), J3.18 (18_GND), J3.21 (21_GND), J3.24 (24_GND), J3.27 (27_GND), J3.3 (3_GND), J3.30 (30_GND), J3.33 (33_GND), J3.5 (5_GND), J3.7 (7_GND), J3.9 (9_GND), R14.2 (B), R15.2 (B), R16.2 (B), R17.2 (B), R18.2 (B), R19.2 (B), SW1.2 (B), SW2.2 (B), U16.3 (GND), U17.4 (GND), U31.5 (GND), U8.4 (GND), MK3.2 (GND), MK4.2 (GND), PCM1.2 (PACK_MINUS), R20.2 (B), U10.3 (GND), U27.5 (GND), U34.5 (GND), U35.4 (GND), U36.3 (GND), Y1.3 (GND); no longer J1.2 (GND), J3.20 (GND), RS8.5 (GND), U16.2 (GND), U17.2 (GND), U31.2 (B), U8.3 (GND)
- net HAPTIC_EN: now also U7.40 (HAPTIC_EN); no longer U7.36 (HAPTIC_EN)
- net I2C_AON_SCL: now also U31.3 (SCL), U8.10 (I2C_SCL), R3.2 (B), U10.4 (SCL), U27.3 (SCL), U35.5 (SCL); no longer R14.2 (B), RS8.3 (SCL), U8.4 (SCL)
- net I2C_AON_SDA: now also U31.4 (SDA), U8.11 (I2C_SDA), R4.2 (B), U10.5 (SDA), U27.4 (SDA), U35.6 (SDA); no longer R15.2 (B), RS8.4 (SDA), U8.5 (SDA)
- net I2S_BCLK: now also U1.40 (I2S_BCLK); no longer U1.36 (I2S_BCLK)
- net I2S_DIN: now also U1.42 (I2S_DIN); no longer U1.38 (I2S_DIN)
- net I2S_LRCLK: now also U1.41 (I2S_LRCLK); no longer U1.37 (I2S_LRCLK)
- net IMU_INT1: now also U7.30 (IMU_INT1), U10.6 (INT1); no longer U7.26 (IMU_INT1), U8.6 (INT1)
- net IMU_INT2: now also U7.31 (IMU_INT2), U10.7 (INT2); no longer U7.27 (IMU_INT2), U8.7 (INT2)
- net NPM_VBAT: now also U8.1 (VBAT), U35.3 (BAT)
- net NRF_SWDCLK: now also U7.42 (SWDCLK); no longer U7.38 (SWDCLK)
- net NRF_SWDIO: now also U7.41 (SWDIO); no longer U7.37 (SWDIO)
- net NTC_L: now also U8.9 (NTC_L), PCM1.5 (NTC2_OR_ID), TP2.5 (NTC_L); no longer RS2.5 (NTC_L)
- net NTC_R: now also U8.8 (NTC_R), PCM1.4 (NTC1), TP2.6 (NTC_R), U35.7 (TS); no longer RS2.6 (NTC_R)
- net PDM_ARRAY_CLK: now also U1.37 (PDM_ARR_CLK), MK3.3 (CLK), MK4.3 (CLK); no longer J3.14 (PDM_ARR_CLK), U1.33 (PDM_ARR_CLK), U16.3 (CLK), U17.3 (CLK)
- net PDM_ARRAY_D0: now also U1.38 (PDM_ARR_D0); no longer J3.15 (PDM_ARR_D0), U1.34 (PDM_ARR_D0)
- net PDM_ARRAY_D1: now also U1.39 (PDM_ARR_D1), MK3.4 (DATA), MK4.4 (DATA); no longer J3.16 (PDM_ARR_D1), U1.35 (PDM_ARR_D1), U16.4 (DATA), U17.4 (DATA)
- net PDM_WAKE_CLK: no longer J3.12 (PDM_WAKE_CLK)
- net PDM_WAKE_DATA: no longer J3.13 (PDM_WAKE_DATA)
- net PMIC_INT_L: now also U8.12 (INT)
- net PMIC_PWRON: now also R12.1 (A); no longer U31.1 (A)
- net PMIC_SHPHLD: now also U8.13 (SHPHLD)
- net SOC_DBG_RX: now also U1.54 (DBG_UART_RX); no longer U1.50 (DBG_UART_RX)
- net SOC_DBG_TX: now also U1.53 (DBG_UART_TX); no longer U1.49 (DBG_UART_TX)
- net SOC_MASKROM_L: now also U1.55 (MASKROM_n); no longer U1.51 (MASKROM_n)
- net SOC_NTC: now also U1.43 (SARADC_NTC); no longer U1.39 (SARADC_NTC)
- net SOC_PMIC_SCL: now also R9.2 (B); no longer R18.2 (B)
- net SOC_PMIC_SDA: now also R10.2 (B); no longer R19.2 (B)
- net SOC_PWRKEY: now also SW1.1 (A), U1.57 (PWRKEY); no longer U1.53 (PWRKEY)
- net SOC_PWR_EN: now also R11.1 (A)
- net SOC_RESET_L: now also SW2.1 (A), U1.56 (RESET_n); no longer U1.52 (RESET_n)
- net SOC_XIN: now also Y1.1 (XIN); no longer U4.1 (XIN)
- net SOC_XOUT: now also Y1.2 (XOUT); no longer U4.2 (XOUT)
- net USB2_DM: now also J1.2 (USB_DN), U1.52 (USB2_DM); no longer J1.4 (DM), U1.48 (USB2_DM)
- net USB2_DP: now also U1.51 (USB2_DP); no longer U1.47 (USB2_DP)
- net USB_5V: now also U8.2 (VBUS), U35.1 (VBUS), U36.2 (OUT); no longer J1.1 (VBUS), J2.1 (VBUS)
- net VCCIO_1V8: now also U4.2 (VCCQ), R10.1 (A), R9.1 (A); no longer R18.1 (A), R19.1 (A)
- net VCC_3V3: now also U4.1 (VCC)
- net VSYS: now also U16.1 (VIN), U8.3 (VSYS), U35.2 (SYS); no longer J3.17 (VSYS)
- net WIFI_BUCK_EN: now also R16.1 (A)
- net WIFI_CHIP_EN: now also R18.1 (A); no longer R11.1 (A)
- net WIFI_LS_EN: now also R17.1 (A)
- net WIFI_PCM_CLK: now also U1.46 (PCM_CLK); no longer U1.42 (PCM_CLK)
- net WIFI_PCM_DIN: now also U1.48 (PCM_DIN); no longer U1.44 (PCM_DIN)
- net WIFI_PCM_DOUT: now also U1.49 (PCM_DOUT); no longer U1.45 (PCM_DOUT)
- net WIFI_PCM_SYNC: now also U1.47 (PCM_SYNC); no longer U1.43 (PCM_SYNC)
- net WIFI_USB_DM: now also U1.45 (USB2_WIFI_DM); no longer U1.41 (USB2_WIFI_DM)
- net WIFI_USB_DP: now also U1.44 (USB2_WIFI_DP); no longer U1.40 (USB2_WIFI_DP)
- net WIFI_WAKE_L: now also U1.50 (WIFI_WAKE_L); no longer U1.46 (WIFI_WAKE_L)
- new net CAM_MODULE_ID: J3.31 (31_MODULE_ID), U14.20 (MODULE_ID)
- new net CHG_CE_L: U35.9 (CE_L), U7.27 (CHG_CE_L)
- new net CHG_INT_L: U35.8 (INT_L), U7.26 (CHG_INT_L)
- new net CHG_PG_L: U35.10 (PG_L), U7.28 (CHG_PG_L)
- new net CSI_D2_N: J3.25 (25_MIPI_D2_N), U1.29 (CSI_D2_N), U14.12 (CSI_D2_N), U34.2 (D2_N)
- new net CSI_D2_P: J3.26 (26_MIPI_D2_P), U1.28 (CSI_D2_P), U14.11 (CSI_D2_P), U34.1 (D2_P)
- new net CSI_D3_N: J3.28 (28_MIPI_D3_N), U1.31 (CSI_D3_N), U14.14 (CSI_D3_N), U34.4 (D3_N)
- new net CSI_D3_P: J3.29 (29_MIPI_D3_P), U1.30 (CSI_D3_P), U14.13 (CSI_D3_P), U34.3 (D3_P)
- new net VBUS_FAULT_L: U36.4 (FLT_L), U7.29 (VBUS_FAULT_L)
- new net VBUS_RAW: J1.5 (VBUS1), J1.6 (VBUS2), J2.1 (VBUS), U36.1 (IN)
- no-connect marks 2 -> 5
Other:
- note added: "AI Glasses V2 (RK3576 Chip-Down) — PRE-LAYOUT SYSTEM SCHEMATIC | 93 components (57 Fit / 18 HOLD / 16 DNP / 2 TBD) | 133 nets | Functional-block capture: power tree + AON control plane + interface buses. Ball-level detail + PCB layout gated behind Gate 0/1/2 (see docs/03_workflow_phases.md). Source: scripts/chipdown_bom.py"
- note removed: "AI Glasses V2 (RK3576 Chip-Down) — PRE-LAYOUT SYSTEM SCHEMATIC | 96 components (58 Fit / 12 HOLD / 19 DNP / 7 TBD) | 127 nets | Functional-block capture: power tree + AON control plane + interface buses. Ball-level detail + PCB layout gated behind Gate 0/1/2 (see docs/03_workflow_phases.md). Source: scripts/chipdown_bom.py"
- moved on the sheet: R11, R12, R13, R14, R15, R16, R17, R18, R19, SW1, SW2, U16
